File: Backplane/Current Control.kicad_sch (KiCad schematic)
At the start: 30 parts, among them Q3 TPHR8504PL,LQ(M1W, Q4 TPHR8504PL,LQ(M1W, U12 LM393, U13 LM358, U15 MCP4725A0T-E/CH, U16 MCP4725A0T-E/CH, U3 LM393, U4 LM358, U8 UCC27324DR

Commit message: Starting to work on layout.
Parts:
- U12, U13, U3, U4: footprint (none) -> COMPONENTS:SOP-8_L4.9-W3.9-P1.27-LS6.0-BL
