File: Backplane/Dual Current Control.kicad_sch (KiCad schematic)
At the start: 28 parts, among them Q25 TPHR8504PL,LQ(M1W, Q26 TPHR8504PL,LQ(M1W, U28 LM393, U29 UCC27324DR, U3 LM358, U32 MCP4725A0T-E/CH, U33 MCP4725A0T-E/CH

Commit message: All parts are correct.
Parts:
- removed unit 2 of U28
- removed unit 1 of U28
- removed U3: LM358, symbol Amplifier_Operational:LM358
- added unit 2 of U1
- added U10: LM393, symbol Comparator:LM393
- added U11, U2: LM358, symbol Amplifier_Operational:LM358
- U1: renamed from U28; footprint COMPONENTS:SOP-8_L4.9-W3.9-P1.27-LS6.0-BL -> (none)
- renumbered C57 to C1, C58 to C2, C52 to C3, C55 to C5, C53 to C6, C54 to C7, C56 to C8, Q25 to Q1, Q26 to Q2, R123 to R1, R131 to R10, R133 to R11, R135 to R12, R129 to R13, R128 to R14, R124 to R2, R125 to R3, R122 to R4, R130 to R5, R132 to R6, R134 to R7, R127 to R8, R126 to R9, U33 to U14, U29 to U7, U32 to U9
Connections:
- net +12V: now also U2.8 (V+)
- net GND: now also U2.4 (V-)
- net at R10.2, R11.1: now also U2.6 (-)
- net at R3.1: now also U10.3 (+)
- net at R2.1: now also U10.2 (-)
- net at Q1.4 (G), R1.2: now also U10.1
- net at Q2.1 (S), Q2.2 (S), Q2.3 (S)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: now also U2.5 (+)
- net at R10.1, R13.2, R8.2: now also U2.7
- net at R14.2, R2.2, R5.1: now also U11.1
- net at Q2.4 (G), R4.2: now also U1.7
- net at R5.2, R6.1: now also U11.2 (-)
- net at Q1.1 (S), Q1.2 (S), Q1.3 (S)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: now also U11.3 (+)
- net at R8.1: now also U1.6 (-)
- net at R9.1: now also U1.5 (+)
