File: Backplane/I2CMux.kicad_sch (KiCad schematic)
At the start: 18 parts, among them U32 TCA9548APWR

Commit message: Starting to work on layout.
Parts:
- renumbered U32 to U14

Commit message: All parts are correct.
Parts:
- renumbered C16 to C9, R56 to R53, R55 to R54, R54 to R55, R53 to R56, R52 to R57, R51 to R58, R50 to R59, R49 to R60, R41 to R61, R42 to R62, R43 to R63, R44 to R64, R45 to R65, R46 to R66, R47 to R67, R48 to R68, U14 to U8
Connections:
- net VCC: now also R56.1
