File: Backplane/PIO_EXT.kicad_sch (KiCad schematic)
At the start: 2 parts, among them U31 PCA9555PW,118

Commit message: Starting to work on layout.
Parts:
- renumbered U31 to U11
Changed lines of the file:
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@@
 		(dnp no)
 		(fields_autoplaced yes)
-		(property "Reference" "U?"
+		(property "Reference" "U11"
 			(at 135.89 45.72 0)
 			(effects
@@
 				)
 				(hide yes)
+			)
+		)
+		(property "Sim.Device" ""
+			(at 135.89 74.93 0)
+			(effects
+				(font
+					(size 1.27 1.27)
+				)
+			)
+		)
+		(property "Sim.Type" ""
+			(at 135.89 74.93 0)
+			(effects
+				(font
+					(size 1.27 1.27)
+				)
 			)
 		)
@@
 				)
 				(path "/4763d09e-4fb7-455a-b785-38411d748b6f/da7544e6-abb6-4349-a9c8-8cf8ece4b836"
-					(reference "U?")
+					(reference "U11")
 					(unit 1)
 				)
@@
 		(dnp no)
 		(fields_autoplaced yes)
-		(property "Reference" "#PWR?"
+		(property "Reference" "#PWR0135"
 			(at 111.76 96.52 0)
 			(effects
@@
 				)
 				(path "/4763d09e-4fb7-455a-b785-38411d748b6f/da7544e6-abb6-4349-a9c8-8cf8ece4b836"
-					(reference "#PWR?")
+					(reference "#PWR0135")
 					(unit 1)
 				)
@@
 			)
 		)
+		(property "Sim.Device" ""
+			(at 110.49 49.53 0)
+			(effects
+				(font
+					(size 1.27 1.27)
+				)
+			)
+		)
+		(property "Sim.Type" ""
+			(at 110.49 49.53 0)
+			(effects
+				(font
+					(size 1.27 1.27)
+				)
+			)
+		)

Commit message: All parts are correct.
Parts:
- renumbered C17 to C8, U11 to U7
Changed lines of the file:
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@@
 		(dnp no)
 		(fields_autoplaced yes)
-		(property "Reference" "U11"
+		(property "Reference" "U7"
 			(at 135.89 45.72 0)
 			(effects
@@
 			(project "Backplane"
 				(path "/4763d09e-4fb7-455a-b785-38411d748b6f/06b95e8c-a01d-4481-87a7-6ca1ab97078e"
-					(reference "U31")
+					(reference "U20")
 					(unit 1)
 				)
 				(path "/4763d09e-4fb7-455a-b785-38411d748b6f/da7544e6-abb6-4349-a9c8-8cf8ece4b836"
-					(reference "U11")
+					(reference "U7")
 					(unit 1)
 				)
@@
 		(dnp no)
 		(fields_autoplaced yes)
-		(property "Reference" "#PWR0135"
+		(property "Reference" "#PWR099"
 			(at 111.76 96.52 0)
 			(effects
@@
 			(project "Backplane"
 				(path "/4763d09e-4fb7-455a-b785-38411d748b6f/06b95e8c-a01d-4481-87a7-6ca1ab97078e"
-					(reference "#PWR0130")
+					(reference "#PWR0146")
 					(unit 1)
 				)
 				(path "/4763d09e-4fb7-455a-b785-38411d748b6f/da7544e6-abb6-4349-a9c8-8cf8ece4b836"
-					(reference "#PWR0135")
+					(reference "#PWR099")
 					(unit 1)
 				)
@@
 		(dnp no)
 		(fields_autoplaced yes)
-		(property "Reference" "#PWR060"
+		(property "Reference" "#PWR098"
 			(at 110.49 39.37 0)
 			(effects
@@
 			(project "Backplane"
 				(path "/4763d09e-4fb7-455a-b785-38411d748b6f/06b95e8c-a01d-4481-87a7-6ca1ab97078e"
-					(reference "#PWR0129")
+					(reference "#PWR0145")
 					(unit 1)
 				)
 				(path "/4763d09e-4fb7-455a-b785-38411d748b6f/da7544e6-abb6-4349-a9c8-8cf8ece4b836"
-					(reference "#PWR060")
+					(reference "#PWR098")
 					(unit 1)
 				)
@@
 		(dnp no)
 		(fields_autoplaced yes)
-		(property "Reference" "C17"
+		(property "Reference" "C8"
 			(at 106.68 50.8001 0)
 			(effects
@@
 			(project "Backplane"
 				(path "/4763d09e-4fb7-455a-b785-38411d748b6f/06b95e8c-a01d-4481-87a7-6ca1ab97078e"
-					(reference "C18")
+					(reference "C22")
 					(unit 1)
 				)
 				(path "/4763d09e-4fb7-455a-b785-38411d748b6f/da7544e6-abb6-4349-a9c8-8cf8ece4b836"
-					(reference "C17")
-					(unit 1)
-				)
+					(reference "C8")
+					(unit 1)
+				)
