File: Backplane/Backplane.kicad_pcb (KiCad board)
At the start: 6 copper layers, 520 x 80 mm, 268 parts, among them J1 Bus_PCI_Express_x1, J2 Bus_PCI_Express_x1, J3 Bus_PCI_Express_x1, J4 Bus_PCI_Express_x1, Q1 CJ2302 S2, Q10 CJ2302 S2, Q11 CJ2302 S2, Q12 CJ2302 S2, Q13 CJ2302 S2, Q14 CJ2302 S2, Q15 CJ2302 S2, Q18 CJ2302 S2, Q19 CJ2302 S2, Q2 CJ2302 S2, Q20 CJ2302 S2, Q21 CJ2302 S2, Q22 CJ2302 S2, Q25 TPHR8504PL,LQ(M1W, Q26 TPHR8504PL,LQ(M1W, Q27 TPHR8504PL,LQ(M1W, Q28 TPHR8504PL,LQ(M1W, Q3 CJ2302 S2, Q4 CJ2302 S2, Q5 CJ2302 S2, Q6 CJ2302 S2, Q7 CJ2302 S2, Q8 CJ2302 S2, Q9 CJ2302 S2, U1 XT60PW-F_C428722, U10 XT60PW-F_C428722, U15 ADS1115IDGSR, U16 ADS1115IDGSR, U17 ADS1115IDGSR, U18 TCA9548APWR, U19 ADS1115IDGSR, U2 XT60PW-F_C428722, U20 PCA9555PW,118, U21 TPS54360BDDAR, U22 TPS54360BDDAR, U23 TPS54360BDDAR, U28 LM393, U29 UCC27324DR, U3 LM358, U32 MCP4725A0T-E/CH, U33 MCP4725A0T-E/CH, U34 LM393, U35 UCC27324DR, U38 MCP4725A0T-E/CH, U39 MCP4725A0T-E/CH, U4 LM358, U7 PCA9555PW,118, U8 TCA9548APWR, U9 XT60PW-F_C428722

Commit message: Layout is almost done.
Parts:
- C19, C58, C59, C60, C61, C62, C63, C64, C65, Q27, Q28, R136, R137, R138, R139, R140, R141, R142, R143, R144, R145, R146, R147, R148, R149, R4, R5, R6, U34, U35, U38, U39, U4: moved to B.Cu
- moved D8 462.6 mm to (97.0, 208.4)
- moved D5 461.7 mm to (89.9, 208.4)
- moved U20 404.2 mm to (137.7, 233.4), turned to -90 degrees
- moved D18 389.8 mm to (70.6, 236.7), turned to -90 degrees
- moved D17 387.2 mm to (75.7, 236.7), turned to -90 degrees
- moved D16 384.7 mm to (80.8, 236.7), turned to -90 degrees
- moved R16 383.2 mm to (70.6, 231.6), turned to 90 degrees
- moved D15 382.2 mm to (85.9, 236.7), turned to -90 degrees
- moved R15 380.5 mm to (75.7, 231.6), turned to 90 degrees
- moved D14 380.0 mm to (91.0, 236.7), turned to -90 degrees
- moved R14 377.9 mm to (80.8, 231.6), turned to 90 degrees
- moved Q10 376.5 mm to (70.6, 226.5), turned to 90 degrees
- moved R13 375.5 mm to (85.9, 231.6), turned to 90 degrees
- moved Q9 373.8 mm to (75.7, 226.5), turned to 90 degrees
- moved R12 373.1 mm to (91.0, 231.6), turned to 90 degrees
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
Commit message: Layout is done.
Parts:
- C18, C23, C24, C25, C26, C27, C28, C29, C30, C31, C32, C33, C34, C35, C36, C37, C38, C39, C40, C41, C42, C43, D1, D2, D29, D3, D30, D31, D4, D5, D6, D7, D8, L1, L2, L3, R100, R101, R102, R103, R104, R105, R106, R107, R108, R109, R110, R111, R112, R22, R23, R24, R25, R26, R27, R28, R29, R30, R31, R32, R33, R99, U21, U22, U23: moved to B.Cu
- moved L3 118.7 mm to (295.5, 197.0), turned to 0 degrees
- moved C40 113.5 mm to (297.3, 204.8), turned to 180 degrees
- moved C43 110.7 mm to (297.3, 208.2), turned to 180 degrees
- moved R3 109.6 mm to (70.0, 226.6)
- moved R4 109.6 mm to (67.7, 226.6)
- moved R5 109.6 mm to (65.4, 226.6)
- moved R6 109.6 mm to (63.1, 226.6)
- moved R1 109.6 mm to (74.6, 226.6)
- moved R2 109.6 mm to (72.3, 226.6)
- moved FPC1 108.5 mm to (65.0, 235.0)
- moved R107 107.8 mm to (283.3, 198.0), turned to 180 degrees
- moved D31 105.6 mm to (290.7, 208.4), turned to -90 degrees
- moved C37 104.4 mm to (282.3, 201.8), turned to 0 degrees
- moved R108 104.2 mm to (278.2, 198.0), turned to 180 degrees
- moved C34 102.4 mm to (282.3, 204.8), turned to 0 degrees
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Routing:
- added copper zone on In1.Cu, net GND
- added copper zone on In4.Cu, net GND
- added copper zone on B.Cu, net GNDPWR
- added copper zone on F.Cu, net GNDPWR
- added copper zone on In1.Cu, net GNDPWR
- added copper zone on In2.Cu, net GNDPWR
- added copper zone on In3.Cu, net GNDPWR
- added copper zone on In4.Cu, net GNDPWR
- added copper zone on B.Cu, net Net-(D29-K)

Commit message: Working on routing.
Parts:
- C19: moved to F.Cu
- moved R31 143.4 mm to (332.4, 208.6)
- moved R32 143.4 mm to (342.5, 208.6)
- moved R33 143.4 mm to (337.4, 208.6)
- moved C21 139.3 mm to (330.1, 200.8), turned to -90 degrees
- moved U19 133.1 mm to (333.4, 200.5), turned to 0 degrees
- moved D4 132.8 mm to (498.5, 203.8), turned to 180 degrees
- moved D1 132.7 mm to (498.5, 207.9), turned to 0 degrees
- moved J1 130.0 mm to (348.7, 200.0)
- moved J2 130.0 mm to (478.7, 200.0)
- moved D6 129.5 mm to (367.6, 202.8), turned to 180 degrees
- moved D7 129.5 mm to (367.6, 206.9), turned to 0 degrees
- moved R30 118.2 mm to (462.4, 208.9)
- moved R28 118.2 mm to (472.5, 208.9)
- moved R29 118.2 mm to (467.5, 208.9)
- moved U17 98.5 mm to (463.7, 200.5), turned to 0 degrees
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Routing:
- net /BatPair2/BatMax - Female1/SDA: track 0.00 -> 126.2 mm, vias 0 -> 1
- net /BatPair2/BatMax - Female1/SCL: track 0.00 -> 112.5 mm, vias 0 -> 1
- net /BAT_LEDS3/LED1: track 0.00 -> 111.1 mm, vias 0 -> 2
- net /BAT_LEDS3/LED2: track 0.00 -> 106.0 mm, vias 0 -> 2
- net /BatPair2/BAT_B_SNS_SDA: track 0.00 -> 103.9 mm, vias 0 -> 3
- net /BatPair2/BAT_B_SNS_SCL: track 0.00 -> 102.2 mm, vias 0 -> 3
- net /BAT_LEDS3/LED3: track 0.00 -> 100.9 mm, vias 0 -> 2
- net /BAT_LEDS3/LED4: track 0.00 -> 96.0 mm, vias 0 -> 2
- net /BAT_LEDS3/LED5: track 0.00 -> 91.1 mm, vias 0 -> 2
- net Net-(U29-OUTA): track 0.00 -> 89.9 mm, vias 0 -> 4
- net Net-(U35-OUTA): track 0.00 -> 86.5 mm, vias 0 -> 4
- net Net-(Q26-G): track 0.00 -> 81.6 mm, vias 0 -> 4
- net /BAT_LEDS4/LED5: track 0.00 -> 78.0 mm, vias 0 -> 2
- net /BAT_LEDS1/LED1: track 0.00 -> 77.2 mm, vias 0 -> 2
- net /BatPair1/ADS1119/A2: track 0.00 -> 75.9 mm, vias 0 -> 1
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- added copper zone on B.Cu, net +12V
- added copper zone on B.Cu, net +24V
- added copper zone on B.Cu, net +48V
- added copper zone on B.Cu, net +5V
- added copper zone on B.Cu, net +BATT
- added copper zone on B.Cu, net /BatPair1/BatMax - Female/P+
- added copper zone on B.Cu, net /BatPair1/BatMax - Female/P-
- added copper zone on B.Cu, net /BatPair1/BatMax - Female1/P+
- added copper zone on B.Cu, net /BatPair1/BatMax - Female1/P-
- added copper zone on B.Cu, net /BatPair2/BatMax - Female/P+
- added copper zone on B.Cu, net /BatPair2/BatMax - Female/P-
- added copper zone on B.Cu, net /BatPair2/BatMax - Female1/P+
- added copper zone on B.Cu, net /BatPair2/BatMax - Female1/P-
- added copper zone on B.Cu, net GND
- added copper zone on B.Cu, net Net-(D30-K)
- added copper zone on B.Cu, net Net-(D31-K)
- added copper zone on B.Cu, net Net-(U3A-+)
- added copper zone on B.Cu, net Net-(U3B-+)
- added copper zone on B.Cu, net Net-(U4A-+)
- added copper zone on B.Cu, net Net-(U4B-+)

Commit message: Almost done routing signals.
Parts:
- moved R134 2.85 mm to (97.9, 185.8), turned to 180 degrees
- moved R111 2.36 mm to (305.7, 165.2), turned to 0 degrees
Routing:
- net /SCL: track 0.00 -> 425.2 mm, vias 0 -> 2
- net /SDA: track 0.00 -> 420.4 mm, vias 0 -> 2
- net /PSUS/EN_BAT_CHG_VLT: track 0.00 -> 255.9 mm, vias 0 -> 5
- net /RESET_A: track 0.00 -> 236.0 mm, vias 0 -> 3
- net /RESET_B: track 0.00 -> 141.2 mm, vias 0 -> 1
- net /BatPair2/BatMax - Female/EEPROM_WC: track 0.00 -> 95.7 mm, vias 0 -> 6
- net /I2CMux1/SDA0: track 11.8 -> 97.2 mm, vias 1 -> 5
- net /I2CMux1/SCL0: track 11.2 -> 96.1 mm, vias 1 -> 5
- net /BatPair2/BAT_A_SNS_ALERT: track 0.00 -> 82.2 mm, vias 0 -> 4
- net /BatPair2/BatMax - Female1/EEPROM_WC: track 0.00 -> 79.3 mm, vias 0 -> 2
- net /BatPair2/BAT_B_SNS_ALERT: track 0.00 -> 78.8 mm, vias 0 -> 2
- net /BatPair2/BatMax - Female/SDA: track 12.8 -> 88.5 mm, vias 1 -> 4
- net /Interrupt_B: track 0.00 -> 68.4 mm, vias 0 -> 3
- net /BatPair2/BatMax - Female/SCL: track 11.3 -> 79.1 mm, vias 1 -> 4
- net /BatPair2/BAT_A_CC_SCL: track 9.05 -> 69.5 mm, vias 1 -> 4
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
Commit message: Routing almost done.
Parts:
- moved R148 3.19 mm to (359.3, 182.2), turned to 180 degrees
Routing:
- net /Interrupt_A: track 10.7 -> 399.7 mm, vias 2 -> 7
- net /RESET_A: track 236.0 -> 396.6 mm, vias 3 -> 5
- net /BatPair1/BatMax - Female1/SDA: track 9.85 -> 143.2 mm, vias 1 -> 4
- net /BatPair1/BatMax - Female1/SCL: track 10.5 -> 129.6 mm, vias 1 -> 3
- net /BatPair1/BAT_B_SNS_ALERT: track 0.00 -> 103.7 mm, vias 0 -> 2
- net /BatPair1/BAT_B_SNS_SCL: track 10.4 -> 110.3 mm, vias 1 -> 3
- net /BatPair1/BatMax - Female1/EEPROM_WC: track 0.00 -> 99.9 mm, vias 0 -> 1
- net /BatPair1/BAT_B_SNS_SDA: track 9.76 -> 108.3 mm, vias 1 -> 3
- net /I2CMux/SDA0: track 11.8 -> 100.8 mm, vias 1 -> 5
- net /I2CMux/SCL0: track 11.2 -> 99.7 mm, vias 1 -> 5
- net /BatPair1/BatMax - Female/SDA: track 11.5 -> 88.9 mm, vias 1 -> 3
- net /BatPair1/BatMax - Female/EEPROM_WC: track 0.00 -> 71.4 mm, vias 0 -> 3
- net /BatPair1/BatMax - Female/SCL: track 10.4 -> 74.1 mm, vias 1 -> 4
- net /BatPair1/BAT_A_SNS_ALERT: track 0.00 -> 63.2 mm, vias 0 -> 4
- net /BatPair1/BAT_A_CC_SCL: track 9.05 -> 60.6 mm, vias 1 -> 4
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