File: Backplane/Backplane.kicad_pcb (KiCad board)
At the start: 6 copper layers, 520 x 80 mm, 271 parts, among them J1 Bus_PCI_Express_x1, J2 Bus_PCI_Express_x1, J3 Bus_PCI_Express_x1, J4 Bus_PCI_Express_x1, Q1 CJ2302 S2, Q10 CJ2302 S2, Q11 CJ2302 S2, Q12 CJ2302 S2, Q13 CJ2302 S2, Q14 CJ2302 S2, Q15 CJ2302 S2, Q18 CJ2302 S2, Q19 CJ2302 S2, Q2 CJ2302 S2, Q20 CJ2302 S2, Q21 CJ2302 S2, Q22 CJ2302 S2, Q25 TPHR8504PL,LQ(M1W, Q26 TPHR8504PL,LQ(M1W, Q27 TPHR8504PL,LQ(M1W, Q28 TPHR8504PL,LQ(M1W, Q3 CJ2302 S2, Q4 CJ2302 S2, Q5 CJ2302 S2, Q6 CJ2302 S2, Q7 CJ2302 S2, Q8 CJ2302 S2, Q9 CJ2302 S2, U1 XT60PW-F_C428722, U10 XT60PW-F_C428722, U15 ADS1115IDGSR, U16 ADS1115IDGSR, U17 ADS1115IDGSR, U18 TCA9548APWR, U19 ADS1115IDGSR, U2 XT60PW-F_C428722, U20 PCA9555PW,118, U21 TPS54360BDDAR, U22 TPS54360BDDAR, U23 TPS54360BDDAR, U28 LM393, U29 UCC27324DR, U3 LM358, U32 MCP4725A0T-E/CH, U33 MCP4725A0T-E/CH, U34 LM393, U35 UCC27324DR, U38 MCP4725A0T-E/CH, U39 MCP4725A0T-E/CH, U4 LM358, U5 AMS1117-3.3_C347222, U7 PCA9555PW,118, U8 TCA9548APWR, U9 XT60PW-F_C428722

Commit message: Update
Parts:
- moved C60 2.05 mm to (407.5, 205.6), turned to 0 degrees
Routing:
- net /Interrupt_A: track 399.9 -> 401.6 mm
- net /Interrupt_B: track 67.8 -> 69.1 mm
- net Net-(Q27-G): track 66.4 -> 65.5 mm
- net /PSUS/EN_BAT_CHG_VLT: track 263.9 -> 264.5 mm
- net Net-(U34B--): track 20.5 -> 20.0 mm
- net GND: vias 337 -> 334
Other:
- board text added: "CX. IN"
- board text added: "INT.A"
- board text added: "INT.B"
- board text added: "RST.A"
- board text added: "RST.B"
- board text added: "SCL"
- board text added: "SDA"
