File: Backplane/PSUS.kicad_sch (KiCad schematic)
At the start: 48 parts, among them U1 XT60PW-F_C428722, U10 XT60PW-F_C428722, U2 XT60PW-F_C428722, U5 TPS54360BDDAR, U6 TPS54360BDDAR, U7 TPS54360BDDAR, U9 XT60PW-F_C428722

Commit message: Update PSUS.kicad_sch
Parts:
- added Q8: TPHR8504PL,LQ(M1W, COMPONENTS:DFN-5_L4.9-W5.9-P1.27-LS6.2-BL, symbol COMPONENTS:TPHR8504PL,LQ(M1W
- added R113: 0, Resistor_SMD:R_1206_3216Metric_Pad1.30x1.75mm_HandSolder, symbol Device:R
- added R114: 200k, Resistor_SMD:R_1206_3216Metric_Pad1.30x1.75mm_HandSolder, symbol Device:R
- added R115: 1k, Resistor_SMD:R_1206_3216Metric_Pad1.30x1.75mm_HandSolder, symbol Device:R
- added R116: 0.001, Resistor_SMD:R_1206_3216Metric_Pad1.30x1.75mm_HandSolder, symbol Device:R
Connections:
- net +48V: now also R113.1; no longer U1.3 (+), U2.3 (+)
- net GND: now also Q8.1 (S), Q8.2 (S), Q8.3 (S), R116.2; no longer U1.4 (-), U10.4 (-), U2.4 (-), U9.4 (-)
- new net: R113.2, R114.1, U1.3 (+), U2.3 (+)
- new net: R114.2, R115.2
- new net: Q8.5 (D), U10.4 (-), U9.4 (-)
- new net: R115.1, R116.1, U1.4 (-), U2.4 (-)

Commit message: Finished board layout.
Parts:
- removed Q8: TPHR8504PL,LQ(M1W, COMPONENTS:DFN-5_L4.9-W5.9-P1.27-LS6.2-BL, symbol COMPONENTS:TPHR8504PL,LQ(M1W
- removed R114: 200k, Resistor_SMD:R_1206_3216Metric_Pad1.30x1.75mm_HandSolder, symbol Device:R
- removed R115: 1k, Resistor_SMD:R_1206_3216Metric_Pad1.30x1.75mm_HandSolder, symbol Device:R
- removed R116: 0.001, Resistor_SMD:R_1206_3216Metric_Pad1.30x1.75mm_HandSolder, symbol Device:R
Connections:
- net GND: now also U1.4 (-), U10.4 (-), U2.4 (-), U9.4 (-)
Other:
- moved on the sheet: R113, U10, U9

Commit message: All parts are correct.
Parts:
- renumbered C8 to C23, C42 to C24, C35 to C25, C29 to C26, C43 to C27, C36 to C28, C30 to C29, C44 to C30, C37 to C31, C31 to C32, C45 to C33, C38 to C34, C32 to C35, C46 to C36, C39 to C37, C33 to C38, C47 to C39, C34 to C41, C48 to C42, C41 to C43, D21 to D29, D23 to D30, D22 to D31, L2 to L1, L4 to L2, R14 to R100, R8 to R101, R5 to R102, R107 to R103, R9 to R104, R6 to R105, R108 to R106, R10 to R107, R12 to R108, R13 to R109, R7 to R110, R11 to R112, R4 to R99, U2 to U1, U9 to U10, U1 to U2, U5 to U21, U7 to U22, U6 to U23, U10 to U9
Connections:
- net EN_BAT_CHG_VLT: now reaches U23.3 (EN)

Commit message: Finished routing.
Parts:
- added C66, C67: 10u, Capacitor_SMD:C_1206_3216Metric, symbol Device:C
- added U5: AMS1117-3.3_C347222, COMPONENTS:SOT-223-4_L6.5-W3.5-P2.30-LS7.0-BR, symbol COMPONENTS:AMS1117-3.3_C347222
Connections:
- net +5V: now also C66.1, U5.3 (VIN)
- net GND: now also C66.2, C67.1, U5.1 (ADJ(GND))
- new net +3.3V: C67.2, U5.2 (VOUT(TAB))
- no-connect marks 8 -> 9
