File: Backplane/Backplane.kicad_sch (KiCad schematic)
At the start: 1 part

Commit message: Starting to work on layout.
Parts:
- added D28, D29, D30, D31, D32, D33, D34, D35: S5BBF, COMPONENTS:SMBF_L4.3-W3.6-LS5.3-RD, symbol COMPONENTS:S5BBF
- added R1, R109, R110, R112, R2, R3: 0, Resistor_SMD:R_1206_3216Metric_Pad1.30x1.75mm_HandSolder, symbol Device:R
Connections:
- net BatPair1/BAT_A+: now also D29.1 (K), D34.2 (A)
- net BatPair1/BAT_B+: now also D28.1 (K), D35.2 (A)
- net BatPair2/BAT_A+: now also D30.1 (K), D32.2 (A)
- net BatPair2/BAT_B+: now also D31.1 (K), D33.2 (A)
- net RESET_A: now also R110.2; no longer FPC1.3
- net RESET_B: now also R2.2; no longer FPC1.4
- net SCL: now also R109.2; no longer FPC1.2
- net SDA: now also R3.2; no longer FPC1.1
- net at FPC1.5: now also R110.1
- net at FPC1.6: now also R112.1
- new net: FPC1.4, R109.1
- new net: FPC1.3, R3.1
- new net: FPC1.1, R1.1
- new net: FPC1.2, R2.1
- new net +24V: D28.2 (A), D29.2 (A), D30.2 (A), D31.2 (A)
- new net +BATT: D32.1 (K), D33.1 (K), D34.1 (K), D35.1 (K)
- new net Interrupt_A: R112.2
- new net Interrupt_B: R1.2
Other:
- added sheet PSUS (PSUS.kicad_sch)

Commit message: All parts are correct.
Parts:
- renumbered D29 to D1, D30 to D2, D32 to D3, D34 to D4, D33 to D5, D35 to D6, D28 to D7, D31 to D8, R109 to R4, R110 to R5, R112 to R6
Connections:
- net PSUS/EN_BAT_CHG_VLT: now reaches FPC1.30
Other:
- sheet BAT_LEDS renamed BAT_LEDS4
- added sheet BAT_LEDS3 (BAT_LEDS.kicad_sch)
- added sheet MountingHoles (MountingHoles.kicad_sch)
- sheet PSUS ports: added EN_BAT_CHG_VLT; removed none

Commit message: added
Parts:
- removed D1, D2, D3, D4, D5, D6, D7, D8: S5BBF, COMPONENTS:SMBF_L4.3-W3.6-LS5.3-RD, symbol COMPONENTS:S5BBF
- removed FPC1: AFC07-S30FCC-00, COMPONENTS:FPC-SMD_P0.50-30P_LCSXJ-H2.0, symbol COMPONENTS:AFC07-S30FCC-00
- removed R1, R2, R3, R4, R5, R6: 0, Resistor_SMD:R_1206_3216Metric_Pad1.30x1.75mm_HandSolder, symbol Device:R
- added U1, U2: XT60PW-F_C428722, COMPONENTS:TH_2P-XT60PW-F, symbol COMPONENTS:XT60PW-F_C428722
Connections:
- net GND: now also U1.4 (-), U2.4 (-)
- new net B+: U1.3 (+), U2.3 (+)
- no-connect marks 2 -> 5
Other:
- removed sheet BAT_LEDS1
- removed sheet BAT_LEDS2
- removed sheet BAT_LEDS3
- removed sheet BAT_LEDS4
- removed sheet I2CMux
- removed sheet I2CMux1
- removed sheet PIO_EXT
- removed sheet PIO_EXT1
- removed sheet PSUS
- sheet BatPair1 ports: added B+, B-; removed BAT_A+, BAT_A_CC_SCL, BAT_A_CC_SDA, BAT_A_CHARGE, BAT_A_EE_SCL, BAT_A_EE_SDA, BAT_A_SNS_ALERT, BAT_A_SNS_SCL, BAT_A_SNS_SDA, BAT_A_WC, BAT_B+, BAT_B_CC_SCL, BAT_B_CC_SDA, BAT_B_CHARGE, BAT_B_EE_SCL, BAT_B_EE_SDA, BAT_B_SNS_ALERT, BAT_B_SNS_SCL, BAT_B_SNS_SDA, BAT_B_WC
- sheet BatPair2 ports: added B+, B-; removed BAT_A+, BAT_A_CC_SCL, BAT_A_CC_SDA, BAT_A_CHARGE, BAT_A_EE_SCL, BAT_A_EE_SDA, BAT_A_SNS_ALERT, BAT_A_SNS_SCL, BAT_A_SNS_SDA, BAT_A_WC, BAT_B+, BAT_B_CC_SCL, BAT_B_CC_SDA, BAT_B_CHARGE, BAT_B_EE_SCL, BAT_B_EE_SDA, BAT_B_SNS_ALERT, BAT_B_SNS_SCL, BAT_B_SNS_SDA, BAT_B_WC
